Commit message: fix: urdf is updates successfully

File: assets/URDF/big_bertha/Spyder_mg995_description.urdf (robot description, URDF)
Before this commit: robot SpdrBot, 17 links, 16 joints
Joints:
- joint Revolute_110: origin xyz=0.06410394 0.07999993 0.04 rpy=1.570796 -0 -0.785 -> xyz=0.07993523 0.06369403 0.04 rpy=1.570796 -0 -0.785
- joint Revolute_113: origin xyz=-0.07989606 0.06299993 0.04 rpy=1.570796 -0 0.785 -> xyz=-0.06357497 0.07983349 0.04 rpy=1.570796 -0 0.785
- joint Revolute_116: origin xyz=-0.06219606 -0.08000007 0.04 rpy=1.570796 -0 2.355 -> xyz=-0.07974269 -0.06374831 0.04 rpy=1.570796 -0 2.355
- joint Revolute_119: origin xyz=0.08010394 -0.06300007 0.04 rpy=1.570796 -0 -2.355 -> xyz=0.06382503 -0.07982906 0.04 rpy=1.570796 -0 -2.355
